File: cerkit48.sch (KiCad schematic (older format))
At the start: 103 parts, among them J1 I2C, SW10 CherryMX, SW11 CherryMX, SW12 CherryMX, SW13 CherryMX, SW14 CherryMX, SW15 CherryMX, SW16 CherryMX, SW17 CherryMX, SW18 CherryMX, SW19 CherryMX, SW2 CherryMX, SW20 CherryMX, SW21 CherryMX, SW22 CherryMX, SW23 CherryMX, SW24 CherryMX, SW25 CherryMX, SW26 CherryMX, SW27 CherryMX, SW28 CherryMX, SW29 CherryMX, SW3 CherryMX, SW30 CherryMX, SW31 CherryMX, SW32 CherryMX, SW33 CherryMX, SW34 CherryMX, SW35 CherryMX, SW36 CherryMX, SW37 CherryMX, SW38 CherryMX, SW39 CherryMX, SW4 CherryMX, SW40 CherryMX, SW41 CherryMX, SW42 CherryMX, SW43 CherryMX, SW44 CherryMX, SW45 CherryMX, SW46 CherryMX, SW47 CherryMX, SW48 CherryMX, SW49 CherryMX, SW5 CherryMX, SW6 CherryMX, SW7 CherryMX, SW8 CherryMX, SW9 CherryMX, U1 proton_c

Commit message: Move proton (#2)
* Move Proton to bottom of board and made board smaller

* Added Proton Pinout diagram

* flipped Proton so it will be arranged correctly on the back of the board.

* Updated reame and fixed stray trace in PCB

* Reworked switches so that they lined up to the grid

* cleaned up PCB

* Update proton-c-pinout_300x300.png

* updated PCB and images

* rounded the edges of the board

* rounded the edges of the PCB

* modified gerber files

* fixed PCB outline
Parts:
- J1: symbol SparkFun-Connectors:CONN_04POLAR -> Connector:Conn_01x04_Male
- U1: footprint proton_c:proton_c -> cerkit48:proton_c_no_center_pins
Connections:
- wire segments 193 -> 190
- no-connect marks 23 -> 16
