File: cerkit48.sch (KiCad schematic (older format))
At the start: 103 parts, among them J1 I2C, SW1 CherryMX, SW10 CherryMX, SW11 CherryMX, SW12 CherryMX, SW13 CherryMX, SW14 CherryMX, SW15 CherryMX, SW16 CherryMX, SW17 CherryMX, SW18 CherryMX, SW19 CherryMX, SW2 CherryMX, SW20 CherryMX, SW21 CherryMX, SW22 CherryMX, SW23 CherryMX, SW24 CherryMX, SW25 CherryMX, SW26 CherryMX, SW27 CherryMX, SW28 CherryMX, SW29 CherryMX, SW3 CherryMX, SW30 CherryMX, SW31 CherryMX, SW32 CherryMX, SW33 CherryMX, SW34 CherryMX, SW35 CherryMX, SW36 CherryMX, SW37 CherryMX, SW38 CherryMX, SW39 CherryMX, SW4 CherryMX, SW40 CherryMX, SW41 CherryMX, SW42 CherryMX, SW43 CherryMX, SW44 CherryMX, SW45 CherryMX, SW46 CherryMX, SW47 CherryMX, SW48 CherryMX, SW5 CherryMX, SW6 CherryMX, SW7 CherryMX, SW8 CherryMX, SW9 CherryMX, U1 proton_c

Commit message: added extra mounting holes and a top and bottom plate
Parts:
- added H? (x3): MountingHole, MountingHole:MountingHole_3.2mm_M3, symbol Mechanical:MountingHole
Changed lines of the file:
@@
 L Mechanical:MountingHole H5
 U 1 1 5F007A46
-P 1500 3200
-F 0 "H5" H 1600 3246 50  0001 L CNN
-F 1 "MountingHole" H 1600 3200 50  0001 L CNN
-F 2 "MountingHole:MountingHole_3.2mm_M3" H 1500 3200 50  0001 C CNN
-F 3 "~" H 1500 3200 50  0001 C CNN
-	1    1500 3200
+P 1850 2200
+F 0 "H5" H 1950 2246 50  0001 L CNN
+F 1 "MountingHole" H 1950 2200 50  0001 L CNN
+F 2 "MountingHole:MountingHole_3.2mm_M3" H 1850 2200 50  0001 C CNN
+F 3 "~" H 1850 2200 50  0001 C CNN
+	1    1850 2200
 	1    0    0    -1
 $EndComp
@@
 L Mechanical:MountingHole H4
 U 1 1 5EFF8634
-P 1500 3000
-F 0 "H4" H 1600 3046 50  0001 L CNN
-F 1 "MountingHole" H 1600 3000 50  0001 L CNN
-F 2 "MountingHole:MountingHole_3.2mm_M3" H 1500 3000 50  0001 C CNN
-F 3 "~" H 1500 3000 50  0001 C CNN
-	1    1500 3000
+P 1850 2000
+F 0 "H4" H 1950 2046 50  0001 L CNN
+F 1 "MountingHole" H 1950 2000 50  0001 L CNN
+F 2 "MountingHole:MountingHole_3.2mm_M3" H 1850 2000 50  0001 C CNN
+F 3 "~" H 1850 2000 50  0001 C CNN
+	1    1850 2000
 	1    0    0    -1
 $EndComp
@@
 L Mechanical:MountingHole H3
 U 1 1 5EFE920E
-P 1500 2800
-F 0 "H3" H 1600 2846 50  0001 L CNN
-F 1 "MountingHole" H 1600 2800 50  0001 L CNN
-F 2 "MountingHole:MountingHole_3.2mm_M3" H 1500 2800 50  0001 C CNN
-F 3 "~" H 1500 2800 50  0001 C CNN
-	1    1500 2800
+P 1850 1800
+F 0 "H3" H 1950 1846 50  0001 L CNN
+F 1 "MountingHole" H 1950 1800 50  0001 L CNN
+F 2 "MountingHole:MountingHole_3.2mm_M3" H 1850 1800 50  0001 C CNN
+F 3 "~" H 1850 1800 50  0001 C CNN
+	1    1850 1800
 	1    0    0    -1
 $EndComp
@@
 L Mechanical:MountingHole H2
 U 1 1 5EFD9E24
-P 1500 2600
-F 0 "H2" H 1600 2646 50  0001 L CNN
-F 1 "MountingHole" H 1600 2600 50  0001 L CNN
-F 2 "MountingHole:MountingHole_3.2mm_M3" H 1500 2600 50  0001 C CNN
-F 3 "~" H 1500 2600 50  0001 C CNN
-	1    1500 2600
+P 1850 1600
+F 0 "H2" H 1950 1646 50  0001 L CNN
+F 1 "MountingHole" H 1950 1600 50  0001 L CNN
+F 2 "MountingHole:MountingHole_3.2mm_M3" H 1850 1600 50  0001 C CNN
+F 3 "~" H 1850 1600 50  0001 C CNN
+	1    1850 1600
 	1    0    0    -1
 $EndComp
@@
 L Mechanical:MountingHole H1
 U 1 1 5EFA9DB5
-P 1500 2400
-F 0 "H1" H 1600 2446 50  0001 L CNN
-F 1 "MountingHole" H 1600 2400 50  0001 L CNN
-F 2 "MountingHole:MountingHole_3.2mm_M3" H 1500 2400 50  0001 C CNN
-F 3 "~" H 1500 2400 50  0001 C CNN
-	1    1500 2400
+P 1850 1400
+F 0 "H1" H 1950 1446 50  0001 L CNN
+F 1 "MountingHole" H 1950 1400 50  0001 L CNN
+F 2 "MountingHole:MountingHole_3.2mm_M3" H 1850 1400 50  0001 C CNN
+F 3 "~" H 1850 1400 50  0001 C CNN
+	1    1850 1400
 	1    0    0    -1
 $EndComp
@@
 Wire Wire Line
 	2200 3750 2200 3900
+$Comp
+L Mechanical:MountingHole H?
+U 1 1 5ED14CA1
+P 1850 2400
+F 0 "H?" H 1950 2446 50  0001 L CNN
+F 1 "MountingHole" H 1950 2400 50  0001 L CNN
+F 2 "MountingHole:MountingHole_3.2mm_M3" H 1850 2400 50  0001 C CNN
+F 3 "~" H 1850 2400 50  0001 C CNN
+	1    1850 2400
+	1    0    0    -1
+$EndComp
+$Comp
+L Mechanical:MountingHole H?
+U 1 1 5ED2282C
+P 1850 2600
+F 0 "H?" H 1950 2646 50  0001 L CNN
+F 1 "MountingHole" H 1950 2600 50  0001 L CNN
+F 2 "MountingHole:MountingHole_3.2mm_M3" H 1850 2600 50  0001 C CNN
+F 3 "~" H 1850 2600 50  0001 C CNN
+	1    1850 2600
+	1    0    0    -1
+$EndComp
+$Comp
+L Mechanical:MountingHole H?
+U 1 1 5ED30330
+P 1850 2800
+F 0 "H?" H 1950 2846 50  0001 L CNN
+F 1 "MountingHole" H 1950 2800 50  0001 L CNN
+F 2 "MountingHole:MountingHole_3.2mm_M3" H 1850 2800 50  0001 C CNN
+F 3 "~" H 1850 2800 50  0001 C CNN
+	1    1850 2800
+	1    0    0    -1
+$EndComp
 $EndSCHEMATC

Commit message: moved controller to the top of the board
Parts:
- removed H2, H3: MountingHole, MountingHole:MountingHole_3.2mm_M3, symbol Mechanical:MountingHole
- gave numbers to parts that had none: 3
Changed lines of the file:
@@
 L Mechanical:MountingHole H5
 U 1 1 5F007A46
-P 1850 2200
-F 0 "H5" H 1950 2246 50  0001 L CNN
-F 1 "MountingHole" H 1950 2200 50  0001 L CNN
-F 2 "MountingHole:MountingHole_3.2mm_M3" H 1850 2200 50  0001 C CNN
-F 3 "~" H 1850 2200 50  0001 C CNN
-	1    1850 2200
+P 2050 2150
+F 0 "H5" H 2150 2196 50  0001 L CNN
+F 1 "MountingHole" H 2150 2150 50  0001 L CNN
+F 2 "MountingHole:MountingHole_3.2mm_M3" H 2050 2150 50  0001 C CNN
+F 3 "~" H 2050 2150 50  0001 C CNN
+	1    2050 2150
 	1    0    0    -1
 $EndComp
@@
 L Mechanical:MountingHole H4
 U 1 1 5EFF8634
-P 1850 2000
-F 0 "H4" H 1950 2046 50  0001 L CNN
-F 1 "MountingHole" H 1950 2000 50  0001 L CNN
-F 2 "MountingHole:MountingHole_3.2mm_M3" H 1850 2000 50  0001 C CNN
-F 3 "~" H 1850 2000 50  0001 C CNN
-	1    1850 2000
-	1    0    0    -1
-$EndComp
-$Comp
-L Mechanical:MountingHole H3
-U 1 1 5EFE920E
-P 1850 1800
-F 0 "H3" H 1950 1846 50  0001 L CNN
-F 1 "MountingHole" H 1950 1800 50  0001 L CNN
-F 2 "MountingHole:MountingHole_3.2mm_M3" H 1850 1800 50  0001 C CNN
-F 3 "~" H 1850 1800 50  0001 C CNN
-	1    1850 1800
-	1    0    0    -1
-$EndComp
-$Comp
-L Mechanical:MountingHole H2
-U 1 1 5EFD9E24
-P 1850 1600
-F 0 "H2" H 1950 1646 50  0001 L CNN
-F 1 "MountingHole" H 1950 1600 50  0001 L CNN
-F 2 "MountingHole:MountingHole_3.2mm_M3" H 1850 1600 50  0001 C CNN
-F 3 "~" H 1850 1600 50  0001 C CNN
-	1    1850 1600
+P 2050 1950
+F 0 "H4" H 2150 1996 50  0001 L CNN
+F 1 "MountingHole" H 2150 1950 50  0001 L CNN
+F 2 "MountingHole:MountingHole_3.2mm_M3" H 2050 1950 50  0001 C CNN
+F 3 "~" H 2050 1950 50  0001 C CNN
+	1    2050 1950
 	1    0    0    -1
 $EndComp
@@
 L Mechanical:MountingHole H1
 U 1 1 5EFA9DB5
-P 1850 1400
-F 0 "H1" H 1950 1446 50  0001 L CNN
-F 1 "MountingHole" H 1950 1400 50  0001 L CNN
-F 2 "MountingHole:MountingHole_3.2mm_M3" H 1850 1400 50  0001 C CNN
-F 3 "~" H 1850 1400 50  0001 C CNN
-	1    1850 1400
+P 2050 1750
+F 0 "H1" H 2150 1796 50  0001 L CNN
+F 1 "MountingHole" H 2150 1750 50  0001 L CNN
+F 2 "MountingHole:MountingHole_3.2mm_M3" H 2050 1750 50  0001 C CNN
+F 3 "~" H 2050 1750 50  0001 C CNN
+	1    2050 1750
 	1    0    0    -1
 $EndComp
@@
 	2200 3750 2200 3900
 $Comp
-L Mechanical:MountingHole H?
+L Mechanical:MountingHole H2
 U 1 1 5ED14CA1
-P 1850 2400
-F 0 "H?" H 1950 2446 50  0001 L CNN
-F 1 "MountingHole" H 1950 2400 50  0001 L CNN
-F 2 "MountingHole:MountingHole_3.2mm_M3" H 1850 2400 50  0001 C CNN
-F 3 "~" H 1850 2400 50  0001 C CNN
-	1    1850 2400
-	1    0    0    -1
-$EndComp
-$Comp
-L Mechanical:MountingHole H?
+P 2050 2350
+F 0 "H2" H 2150 2396 50  0001 L CNN
+F 1 "MountingHole" H 2150 2350 50  0001 L CNN
+F 2 "MountingHole:MountingHole_3.2mm_M3" H 2050 2350 50  0001 C CNN
+F 3 "~" H 2050 2350 50  0001 C CNN
+	1    2050 2350
+	1    0    0    -1
+$EndComp
+$Comp
+L Mechanical:MountingHole H3
 U 1 1 5ED2282C
-P 1850 2600
-F 0 "H?" H 1950 2646 50  0001 L CNN
-F 1 "MountingHole" H 1950 2600 50  0001 L CNN
-F 2 "MountingHole:MountingHole_3.2mm_M3" H 1850 2600 50  0001 C CNN
-F 3 "~" H 1850 2600 50  0001 C CNN
-	1    1850 2600
-	1    0    0    -1
-$EndComp
-$Comp
-L Mechanical:MountingHole H?
+P 2050 2550
+F 0 "H3" H 2150 2596 50  0001 L CNN
+F 1 "MountingHole" H 2150 2550 50  0001 L CNN
+F 2 "MountingHole:MountingHole_3.2mm_M3" H 2050 2550 50  0001 C CNN
+F 3 "~" H 2050 2550 50  0001 C CNN
+	1    2050 2550
+	1    0    0    -1
+$EndComp
+$Comp
+L Mechanical:MountingHole H6
 U 1 1 5ED30330
-P 1850 2800
-F 0 "H?" H 1950 2846 50  0001 L CNN
-F 1 "MountingHole" H 1950 2800 50  0001 L CNN
-F 2 "MountingHole:MountingHole_3.2mm_M3" H 1850 2800 50  0001 C CNN
-F 3 "~" H 1850 2800 50  0001 C CNN
-	1    1850 2800
-	1    0    0    -1
-$EndComp
+P 2050 2750
+F 0 "H6" H 2150 2796 50  0001 L CNN
+F 1 "MountingHole" H 2150 2750 50  0001 L CNN
+F 2 "MountingHole:MountingHole_3.2mm_M3" H 2050 2750 50  0001 C CNN
+F 3 "~" H 2050 2750 50  0001 C CNN
+	1    2050 2750
+	1    0    0    -1
+$EndComp
