File: cerkit48.kicad_pcb (KiCad board)
At the start: 2 copper layers, 236.5 x 84.1 mm, 103 parts, among them J1 I2C, SW1 CherryMX, SW10 CherryMX, SW11 CherryMX, SW12 CherryMX, SW13 CherryMX, SW14 CherryMX, SW15 CherryMX, SW16 CherryMX, SW17 CherryMX, SW18 CherryMX, SW19 CherryMX, SW2 CherryMX, SW20 CherryMX, SW21 CherryMX, SW22 CherryMX, SW23 CherryMX, SW24 CherryMX, SW25 CherryMX, SW26 CherryMX, SW27 CherryMX, SW28 CherryMX, SW29 CherryMX, SW3 CherryMX, SW30 CherryMX, SW31 CherryMX, SW32 CherryMX, SW33 CherryMX, SW34 CherryMX, SW35 CherryMX, SW36 CherryMX, SW37 CherryMX, SW38 CherryMX, SW39 CherryMX, SW4 CherryMX, SW40 CherryMX, SW41 CherryMX, SW42 CherryMX, SW43 CherryMX, SW44 CherryMX, SW45 CherryMX, SW46 CherryMX, SW47 CherryMX, SW48 CherryMX, SW5 CherryMX, SW6 CherryMX, SW7 CherryMX, SW8 CherryMX, SW9 CherryMX, U1 proton_c

Commit message: added extra mounting holes and a top and bottom plate
Parts:
- added H6: MountingHole, MountingHole:MountingHole_3.2mm_M3, F.Cu at (102.2, 134.7)
- added H7: MountingHole, MountingHole:MountingHole_3.2mm_M3, F.Cu at (180.4, 134.7)
- added H8: MountingHole, MountingHole:MountingHole_3.2mm_M3, F.Cu at (258.6, 134.7)
- moved H4 244.8 mm to (258.6, 52.5)
- moved H5 231.6 mm to (24.0, 134.7)
- moved H2 153.4 mm to (102.2, 52.5)
- moved H3 56.8 mm to (180.4, 52.5)
- moved H1 4.22 mm to (24.0, 52.5)
Routing:
- removed copper zone on B.Cu, net GND
- removed copper zone on F.Cu, net GND
Other:
- board size 236.5 x 84.1 mm -> 240.7 x 88.3 mm
